Commit message: Add collision disable macros and use

File: vigir_atlas_moveit_config/config/vigir_atlas.srdf.xacro (robot description, xacro)
@@ -11,21 +11,21 @@
   <xacro:include filename="$(find flor_atlas_moveit_config)/config/multisense/$(env FLOR_MULTISENSE_TYPE).srdf.xacro" />-->
   <!--Create macro that will be used to disable collisions for links that lie inside other collision geometry below-->
-<!--  <xacro:macro name="disable_all_collisions" params="disable_link_name">
+  <xacro:macro name="disable_all_collisions" params="disable_link_name">
     <xacro:disable_robot_collision_helper disable_robot_link_name="${disable_link_name}"/>
-    <xacro:disable_left_hand_collision_checks link_name="${disable_link_name}"/>
+<!--    <xacro:disable_left_hand_collision_checks link_name="${disable_link_name}"/>
     <xacro:disable_right_hand_collision_checks link_name="${disable_link_name}"/>
-    <xacro:disable_multisense_collision_helper link_name="${disable_link_name}"/>
+    <xacro:disable_multisense_collision_helper link_name="${disable_link_name}"/>-->
   </xacro:macro>
-  <xacro:disable_all_collisions disable_link_name="ltorso" />
-  <xacro:disable_all_collisions disable_link_name="mtorso" />
+<!--  <xacro:disable_all_collisions disable_link_name="ltorso" />
+  <xacro:disable_all_collisions disable_link_name="mtorso" />-->
   <xacro:disable_all_collisions disable_link_name="hokuyo_link" />
   <xacro:disable_all_collisions disable_link_name="l_situational_awareness_camera_link" />
   <xacro:disable_all_collisions disable_link_name="r_situational_awareness_camera_link" />
-  <xacro:disable_all_collisions disable_link_name="l_uglut" />
+<!--  <xacro:disable_all_collisions disable_link_name="l_uglut" />
   <xacro:disable_all_collisions disable_link_name="r_uglut" />
   <xacro:disable_all_collisions disable_link_name="l_lglut" />
   <xacro:disable_all_collisions disable_link_name="r_lglut" />
   <xacro:disable_all_collisions disable_link_name="l_talus" />
-  <xacro:disable_all_collisions disable_link_name="r_talus" />
+  <xacro:disable_all_collisions disable_link_name="r_talus" />-->
   <xacro:disable_all_collisions disable_link_name="imu_link" />-->
   <!--Disable to be able to close gap between pelvis and utorso-->
