Commit message: Changed robotiq joint types to mimic

File: vigir_atlas_moveit_config/config/hands/l_robotiq.srdf.xacro (robot description, xacro)
@@ -7,11 +7,4 @@
       <joint name="left_f2_j1" />
       <joint name="left_f1_j0" />
-      <joint name="left_f2_j0" />
-      <joint name="left_f0_j2" />
-      <joint name="left_f1_j2" />
-      <joint name="left_f2_j2" />
-      <joint name="left_f0_j3" />
-      <joint name="left_f1_j3" />
-      <joint name="left_f2_j3" />
   </group>
   <end_effector name="l_hand_eef" parent_link="l_hand" group="left_hand" />

File: vigir_atlas_moveit_config/config/hands/r_robotiq.srdf.xacro (robot description, xacro)
@@ -7,11 +7,4 @@
       <joint name="right_f2_j1" />
       <joint name="right_f1_j0" />
-      <joint name="right_f2_j0" />
-      <joint name="right_f0_j2" />
-      <joint name="right_f1_j2" />
-      <joint name="right_f2_j2" />
-      <joint name="right_f0_j3" />
-      <joint name="right_f1_j3" />
-      <joint name="right_f2_j3" />
   </group>
   <end_effector name="r_hand_eef" parent_link="r_hand" group="right_hand" />

Commit message: Added underactuated joints to srdf

File: vigir_atlas_moveit_config/config/hands/l_robotiq.srdf.xacro (robot description, xacro)
@@ -7,4 +7,11 @@
       <joint name="left_f2_j1" />
       <joint name="left_f1_j0" />
+      <joint name="left_f2_j0" />
+      <joint name="left_f0_j2" />
+      <joint name="left_f1_j2" />
+      <joint name="left_f2_j2" />
+      <joint name="left_f0_j3" />
+      <joint name="left_f1_j3" />
+      <joint name="left_f2_j3" />
   </group>
   <end_effector name="l_hand_eef" parent_link="l_hand" group="left_hand" />

File: vigir_atlas_moveit_config/config/hands/r_robotiq.srdf.xacro (robot description, xacro)
@@ -7,4 +7,11 @@
       <joint name="right_f2_j1" />
       <joint name="right_f1_j0" />
+      <joint name="right_f2_j0" />
+      <joint name="right_f0_j2" />
+      <joint name="right_f1_j2" />
+      <joint name="right_f2_j2" />
+      <joint name="right_f0_j3" />
+      <joint name="right_f1_j3" />
+      <joint name="right_f2_j3" />
   </group>
   <end_effector name="r_hand_eef" parent_link="r_hand" group="right_hand" />

Commit message: Added group for active hand joints

File: vigir_atlas_moveit_config/config/hands/l_robotiq.srdf.xacro (robot description, xacro)
@@ -15,4 +15,10 @@
       <joint name="left_f2_j3" />
   </group>
+  <group name="active_left_hand">
+      <joint name="left_f0_j1" />
+      <joint name="left_f1_j1" />
+      <joint name="left_f2_j1" />
+      <joint name="left_f1_j0" />
+  </group>
   <end_effector name="l_hand_eef" parent_link="l_hand" group="left_hand" />
   <xacro:disable_robotiq_hand_self_collisions side="left"/>

File: vigir_atlas_moveit_config/config/hands/r_robotiq.srdf.xacro (robot description, xacro)
@@ -15,4 +15,10 @@
       <joint name="right_f2_j3" />
   </group>
+  <group name="active_right_hand">
+      <joint name="right_f0_j1" />
+      <joint name="right_f1_j1" />
+      <joint name="right_f2_j1" />
+      <joint name="right_f1_j0" />
+  </group>
   <end_effector name="r_hand_eef" parent_link="r_hand" group="right_hand" />
   <xacro:disable_robotiq_hand_self_collisions side="right"/>
